Commit message: Major update to the Roomba ROS metapackage.

File: roomba_description/urdf/black_roomba.urdf.xacro (robot description, xacro)
@@ -138,30 +138,30 @@
 	</link>
 	<joint name="left_ir_sensor_joint" type="fixed">
+	  	<origin xyz="0.01 0.15 0.042" rpy="0 0 1.5" />
+	    	<parent link="base_link"/>
+	    	<child link="left_ir_sensor_link" />
+	</joint>
+	<joint name="front_left_ir_sensor_joint" type="fixed">
+	  	<origin xyz="0.09 0.12 0.042" rpy="0 0 1.0" />
+	    	<parent link="base_link"/>
+	    	<child link="front_left_ir_sensor_link" />
+	</joint>
+	<joint name="center_left_ir_sensor_joint" type="fixed">
+	  	<origin xyz="0.15 0.04 0.042" rpy="0 0 0.4" />
+	    	<parent link="base_link"/>
+	    	<child link="center_left_ir_sensor_link" />
+	</joint>
+	<joint name="center_right_ir_sensor_joint" type="fixed">
+	  	<origin xyz="0.15 -0.04 0.042" rpy="0 0 -0.4" />
+	    	<parent link="base_link"/>
+	    	<child link="center_right_ir_sensor_link" />
+	</joint>
+	<joint name="front_right_ir_sensor_joint" type="fixed">
+	  	<origin xyz="0.09 -0.120 0.042" rpy="0 0 -1.0" />
+	    	<parent link="base_link"/>
+	    	<child link="front_right_ir_sensor_link" />
+	</joint>
+	<joint name="right_ir_sensor_joint" type="fixed">
 	  	<origin xyz="0.01 -0.15 0.042" rpy="0 0 -1.5" />
-	    	<parent link="base_link"/>
-	    	<child link="left_ir_sensor_link" />
-	</joint>
-	<joint name="front_left_ir_sensor_joint" type="fixed">
-	  	<origin xyz="0.09 -0.12 0.042" rpy="0 0 -1.0" />
-	    	<parent link="base_link"/>
-	    	<child link="front_left_ir_sensor_link" />
-	</joint>
-	<joint name="center_left_ir_sensor_joint" type="fixed">
-	  	<origin xyz="0.15 -0.04 0.042" rpy="0 0 -0.4" />
-	    	<parent link="base_link"/>
-	    	<child link="center_left_ir_sensor_link" />
-	</joint>
-	<joint name="center_right_ir_sensor_joint" type="fixed">
-	  	<origin xyz="0.15 0.04 0.042" rpy="0 0 0.4" />
-	    	<parent link="base_link"/>
-	    	<child link="center_right_ir_sensor_link" />
-	</joint>
-	<joint name="front_right_ir_sensor_joint" type="fixed">
-	  	<origin xyz="0.09 0.120 0.042" rpy="0 0 1.0" />
-	    	<parent link="base_link"/>
-	    	<child link="front_right_ir_sensor_link" />
-	</joint>
-	<joint name="right_ir_sensor_joint" type="fixed">
-	  	<origin xyz="0.01 0.15 0.042" rpy="0 0 1.5" />
 	    	<parent link="base_link"/>
 	    	<child link="right_ir_sensor_link" />

File: roomba_description/urdf/white_roomba.urdf.xacro (robot description, xacro)
@@ -138,30 +138,30 @@
 	</link>
 	<joint name="left_ir_sensor_joint" type="fixed">
+	  	<origin xyz="0.01 0.15 0.042" rpy="0 0 1.5" />
+	    	<parent link="base_link"/>
+	    	<child link="left_ir_sensor_link" />
+	</joint>
+	<joint name="front_left_ir_sensor_joint" type="fixed">
+	  	<origin xyz="0.09 0.12 0.042" rpy="0 0 1.0" />
+	    	<parent link="base_link"/>
+	    	<child link="front_left_ir_sensor_link" />
+	</joint>
+	<joint name="center_left_ir_sensor_joint" type="fixed">
+	  	<origin xyz="0.15 0.04 0.042" rpy="0 0 0.4" />
+	    	<parent link="base_link"/>
+	    	<child link="center_left_ir_sensor_link" />
+	</joint>
+	<joint name="center_right_ir_sensor_joint" type="fixed">
+	  	<origin xyz="0.15 -0.04 0.042" rpy="0 0 -0.4" />
+	    	<parent link="base_link"/>
+	    	<child link="center_right_ir_sensor_link" />
+	</joint>
+	<joint name="front_right_ir_sensor_joint" type="fixed">
+	  	<origin xyz="0.09 -0.120 0.042" rpy="0 0 -1.0" />
+	    	<parent link="base_link"/>
+	    	<child link="front_right_ir_sensor_link" />
+	</joint>
+	<joint name="right_ir_sensor_joint" type="fixed">
 	  	<origin xyz="0.01 -0.15 0.042" rpy="0 0 -1.5" />
-	    	<parent link="base_link"/>
-	    	<child link="left_ir_sensor_link" />
-	</joint>
-	<joint name="front_left_ir_sensor_joint" type="fixed">
-	  	<origin xyz="0.09 -0.12 0.042" rpy="0 0 -1.0" />
-	    	<parent link="base_link"/>
-	    	<child link="front_left_ir_sensor_link" />
-	</joint>
-	<joint name="center_left_ir_sensor_joint" type="fixed">
-	  	<origin xyz="0.15 -0.04 0.042" rpy="0 0 -0.4" />
-	    	<parent link="base_link"/>
-	    	<child link="center_left_ir_sensor_link" />
-	</joint>
-	<joint name="center_right_ir_sensor_joint" type="fixed">
-	  	<origin xyz="0.15 0.04 0.042" rpy="0 0 0.4" />
-	    	<parent link="base_link"/>
-	    	<child link="center_right_ir_sensor_link" />
-	</joint>
-	<joint name="front_right_ir_sensor_joint" type="fixed">
-	  	<origin xyz="0.09 0.120 0.042" rpy="0 0 1.0" />
-	    	<parent link="base_link"/>
-	    	<child link="front_right_ir_sensor_link" />
-	</joint>
-	<joint name="right_ir_sensor_joint" type="fixed">
-	  	<origin xyz="0.01 0.15 0.042" rpy="0 0 1.5" />
 	    	<parent link="base_link"/>
 	    	<child link="right_ir_sensor_link" />
@@ -204,5 +204,5 @@
 	        		<cylinder radius="0.033" length = "0.023"/>
 	      		</geometry>
-			<material name="Gray" />
+			<material name="DarkGray" />
 	    	</visual>
 	    	<collision>
@@ -230,5 +230,5 @@
 	        		<cylinder radius="0.033" length = "0.023"/>
 	      		</geometry>
-			<material name="Gray" />
+			<material name="DarkGray" />
 	    	</visual>
 	  	<collision>
@@ -257,5 +257,5 @@
 				<sphere radius="0.018" />
 	      		</geometry>
-			<material name="Gray" />
+			<material name="DarkGray" />
 	    	</visual>
 	    	<collision>
