Commit message: Combined black & white urdf files into a single urdf file which takes color as a parameter.  Launch files updated accordingly.

File: roomba_description/urdf/roomba.urdf.xacro (robot description, xacro)
@@ -30,5 +30,5 @@
 	      		<origin xyz=" 0 0 0.0308" rpy="0 0 1.5708" />
 	      		<geometry>
-	        		<mesh filename="package://roomba_description/meshes/black_roomba.dae"/>
+	        		<mesh filename="package://roomba_description/meshes/$(arg color)_roomba.dae"/>
 	      		</geometry>
 	    	</visual>

Commit message: fixed size of collision cylinder for base_link.  Radius increased by a power of 10, length approximated 2 cm taller than it was

File: roomba_description/urdf/roomba.urdf.xacro (robot description, xacro)
@@ -36,5 +36,5 @@
 	      		<origin xyz="0.0 0.0 0.0308" rpy="0 0 0" />
 	      		<geometry>
-	        		<cylinder length="0.0611632" radius="0.016495"/>
+	        		<cylinder length="0.0811632" radius="0.16495"/>
 	     	 	</geometry>
 	    	</collision>

Commit message: base_footprint now has the collision properties of circle the radius of the roomba, with no height.  The visual properties have been removed (because they confuse the visual model. Also tweeked the collision properties of the base_link again

File: roomba_description/urdf/roomba.urdf.xacro (robot description, xacro)
@@ -6,16 +6,9 @@
 	<!-- base_footprint is a fictitious link(frame) that is on the ground right below base_link origin, navigation stack depends on this frame -->
 	<link name="base_footprint">
-		<visual>
-	  		<origin xyz="0 0 0" rpy="0 0 0" />
-	      		<geometry>
-	        		<box size="0.001 0.001 0.001" />
-	      		</geometry>
-			<material name="Green" />
-	 	</visual>
 	 	<collision>
-	      		<origin xyz="0 0 0.017" rpy="0 0 0" />
-	      		<geometry>
-	       			<box size="0.001 0.001 0.001" />
-	      		</geometry>
+	      		<origin xyz="0 0 0" rpy="0 0 0" />
+	      		<geometry>
+	        		<cylinder length="0" radius="0.16495"/>
+	     	 	</geometry>
 	    	</collision>
 	</link>
@@ -34,7 +27,7 @@
 	    	</visual>
 	    	<collision>
-	      		<origin xyz="0.0 0.0 0.0308" rpy="0 0 0" />
-	      		<geometry>
-	        		<cylinder length="0.0811632" radius="0.16495"/>
+	      		<origin xyz="0.0 0.0 0.0358" rpy="0 0 0" />
+	      		<geometry>
+	        		<cylinder length="0.0711632" radius="0.16495"/>
 	     	 	</geometry>
 	    	</collision>
